Commit message: Copy fake joints and links also to the simplified model

File: urdf/ergoCub/robots/handMK5SimplifiedGazeboV1/model.urdf (robot description, URDF)
Before this commit: robot ergoCub, 14 links, 13 joints
Links:
- added link l_hand_palm_shifted, mass 0.1
- added link study_center, mass 0.1
Joints:
- added joint l_thumb_1_study_rotation: type revolute, parent l_hand_thumb_1, child study_center, origin xyz=-0.0016246634  0.0025732007  0.0035903516 rpy=0.0000003279 0.2268932149 0.3946688174, axis 0.0 -1.0 0.0, limit lower=0.0 upper=1.57 effort=50000 velocity=0.0
- added joint l_thumb_1_study_translation: type prismatic, parent l_hand_palm, child l_hand_palm_shifted, origin xyz=0.0 0.0 0.0 rpy=0.0 0.0 0.0, axis 0.0 0.0 -1.0, limit lower=-0.04 upper=0.04 effort=50000 velocity=0.1
- joint l_thumb_add: parent l_hand_palm -> l_hand_palm_shifted
- joint l_thumb_prox: parent l_hand_thumb_1 -> study_center
