Commit message: Release all limits within the URDF to ease tests

File: urdf/ergoCub/robots/handMK5GazeboV1/model.urdf (robot description, URDF)
Before this commit: robot ergoCub, 14 links, 13 joints
Joints:
- joint l_index_add: limit lower=0.0 upper=0.3490658503988659 effort=50000 velocity=120.0 -> lower=0.0 upper=3.14 effort=50000 velocity=120.0
- joint l_index_dist: limit lower=0.0 upper=2.792526803190927 effort=50000 velocity=120.0 -> lower=0.0 upper=3.14 effort=50000 velocity=120.0
- joint l_index_prox: limit lower=0.0 upper=2.792526803190927 effort=50000 velocity=120.0 -> lower=0.0 upper=3.14 effort=50000 velocity=120.0
- joint l_thumb_add: limit lower=0.0 upper=1.0471975511965976 effort=50000 velocity=120.0 -> lower=0.0 upper=3.14 effort=50000 velocity=120.0

Commit message: Add fake links so that the link of the hand palm is standalone

File: urdf/ergoCub/robots/handMK5GazeboV1/model.urdf (robot description, URDF)
Before this commit: robot ergoCub, 14 links, 13 joints
Links:
- link root_link: mass None -> 1.0
Joints:
- joint base_link_fixed_joint: limit (none) -> lower=0.0 upper=0.0 effort=50000 velocity=0.0; type fixed -> revolute

File: urdf/ergoCub/robots/handMK5SimplifiedGazeboV1/model.urdf (robot description, URDF)
Before this commit: robot ergoCub, 14 links, 13 joints
Links:
- link root_link: mass None -> 1.0
Joints:
- joint base_link_fixed_joint: limit (none) -> lower=0.0 upper=0.0 effort=50000 velocity=0.0; type fixed -> revolute

Commit message: Add fake reference frame containing the center of rotation for the thumb modification

File: urdf/ergoCub/robots/handMK5GazeboV1/model.urdf (robot description, URDF)
Before this commit: robot ergoCub, 14 links, 13 joints
Links:
- added link study_center, mass 1.0
Joints:
- added joint hand_palm_study_center_joint: type revolute, parent l_hand_palm, child study_center, origin xyz= 0.0220700000  0.0000000000 -0.0311400000 rpy= 0.0000000000 -0.0000000000  0.0000000000, axis 1.0 0.0 0.0, limit lower=0.0 upper=0.0 effort=50000 velocity=0.0

Commit message: Implement a fake actuated joint that allows rotating the thumb assembly around the point provided in https://github.com/icub-tech-iit/ergocub-design-lowerarm/issues/131#issuecomment-1481006986

File: urdf/ergoCub/robots/handMK5GazeboV1/model.urdf (robot description, URDF)
Before this commit: robot ergoCub, 15 links, 14 joints
Joints:
- added joint l_thumb_1_study_center: type revolute, parent l_hand_thumb_1, child study_center, origin xyz=-0.0016246634  0.0025732007  0.0035903516 rpy=0.0000003279 0.2268932149 0.3946688174, axis 0.0 -1.0 0.0, limit lower=0.0 upper=1.57 effort=50000 velocity=0.0
- joint l_thumb_prox: origin xyz=0.03454190438141733 0.0031447987794122334 -0.026071809138455138 rpy=1.3486854426081958 0.6514100961972398 1.2371890149379312e-06 -> xyz= 0.0394172294 -0.0133784864 -0.0213421944 rpy=-1.6971767845  2.7019317802  2.7969048054; parent l_hand_thumb_1 -> study_center

Commit message: Implement a fake actuated joint that allows translating the thum assembly along the z axis of the hand palm frame

File: urdf/ergoCub/robots/handMK5GazeboV1/model.urdf (robot description, URDF)
Before this commit: robot ergoCub, 15 links, 15 joints
Links:
- added link l_hand_palm_shifted, mass 0.1
- link study_center: mass 1.0 -> 0.1
Joints:
- removed joint l_thumb_1_study_center
- added joint l_thumb_1_study_rotation: type revolute, parent l_hand_thumb_1, child study_center, origin xyz=-0.0016246634  0.0025732007  0.0035903516 rpy=0.0000003279 0.2268932149 0.3946688174, axis 0.0 -1.0 0.0, limit lower=0.0 upper=1.57 effort=50000 velocity=0.0
- added joint l_thumb_1_study_translation: type prismatic, parent l_hand_palm, child l_hand_palm_shifted, origin xyz=0.0 0.0 0.0 rpy=0.0 0.0 0.0, axis 0.0 0.0 -1.0, limit lower=-0.04 upper=0.04 effort=50000 velocity=0.1
- joint hand_palm_study_center_joint: parent l_hand_palm -> l_hand_palm_shifted
- joint l_thumb_add: parent l_hand_palm -> l_hand_palm_shifted

Commit message: Update implementation of fake joints

File: urdf/ergoCub/robots/handMK5GazeboV1/model.urdf (robot description, URDF)
Before this commit: robot ergoCub, 16 links, 16 joints
Links:
- removed link l_hand_palm_shifted
- removed link study_center
- added link l_hand_thumb_1_pivot, mass 0.1
Joints:
- removed joint hand_palm_study_center_joint
- removed joint l_thumb_1_study_rotation
- removed joint l_thumb_1_study_translation
- added joint l_thumb_pivot: type revolute, parent l_hand_thumb_1, child l_hand_thumb_1_pivot, origin xyz=0.0000000000 0.0000000000 0.0052300000 rpy=-1.5707963268  0.0000000000  0.2201356130, axis 0.0 0.0 -1.0, limit lower=0.0 upper=1.5707963267948966 effort=50000 velocity=100.0
- joint l_thumb_add: parent l_hand_palm_shifted -> l_hand_palm
- joint l_thumb_prox: origin xyz= 0.0394172294 -0.0133784864 -0.0213421944 rpy=-1.6971767845  2.7019317802  2.7969048054 -> xyz= 0.0343950383  0.0313018091 -0.0044737301 rpy=3.0543263593 0.1745316748 0.6632251552; parent study_center -> l_hand_thumb_1_pivot

Commit message: Disable visualization of l_hand_thumb_1

File: urdf/ergoCub/robots/handMK5GazeboV1/model.urdf (robot description, URDF)
Before this commit: robot ergoCub, 15 links, 14 joints
Links:
- link l_hand_thumb_1: geometry 

Commit message: Add fake joints required to study thumb proximal length in relationship with a change of the thumb attachment point to the palm

File: urdf/ergoCub/robots/handMK5GazeboV1/model.urdf (robot description, URDF)
Before this commit: robot ergoCub, 15 links, 14 joints
Links:
- added link l_hand_thumb_2_down_shifter, mass 0.1
- added link l_hand_thumb_2_up_shifter, mass 0.1
Joints:
- added joint l_thumb_down_shifter: type prismatic, parent l_hand_thumb_1_pivot, child l_hand_thumb_2_down_shifter, origin xyz= 0.0343950383  0.0313018091 -0.0044737301 rpy=3.0543263593 0.1745316748 0.6632251552, axis -1.0 0.0 0.0, limit lower=0.0 upper=0.03 effort=50000 velocity=0.1
- added joint l_thumb_shifter_coupled: type prismatic, parent l_hand_thumb_2, child l_hand_thumb_2_up_shifter, origin xyz=0.01999951842714734 -0.0014995220956423305 4.0850220001109605e-07 rpy=0.0 0.0 0.0, axis 1.0 0.0 0.0, limit lower=0.0 upper=0.03 effort=50000 velocity=0.1
- joint l_thumb_dist: origin xyz=0.01999951842714734 -0.0014995220956423305 4.0850220001109605e-07 rpy=0 0 0 -> xyz=0.0 0.0 0.0 rpy=0.0 0.0 0.0; parent l_hand_thumb_2 -> l_hand_thumb_2_up_shifter
- joint l_thumb_prox: origin xyz= 0.0343950383  0.0313018091 -0.0044737301 rpy=3.0543263593 0.1745316748 0.6632251552 -> xyz=0.0 0.0 0.0 rpy=0.0 0.0 0.0; parent l_hand_thumb_1_pivot -> l_hand_thumb_2_down_shifter

Commit message: Add fake joints required to study fingers length

File: urdf/ergoCub/robots/handMK5GazeboV1/model.urdf (robot description, URDF)
Before this commit: robot ergoCub, 17 links, 16 joints
Links:
- added link l_hand_index_2_shifter, mass 0.1
- added link l_hand_index_3_shifter, mass 0.1
- added link l_hand_middle_1_shifter, mass 0.1
- added link l_hand_middle_2_shifter, mass 0.1
- added link l_hand_pinkie_1_shifter, mass 0.1
- added link l_hand_pinkie_2_shifter, mass 0.1
- added link l_hand_ring_1_shifter, mass 0.1
- added link l_hand_ring_2_shifter, mass 0.1
Joints:
- added joint l_index_2_shifter: type prismatic, parent l_hand_index_2, child l_hand_index_2_shifter, origin xyz=0 -0.0015006327879180659 -0.02999922319857601 rpy=0 0 0, axis 0.0 0.0 -1.0, limit lower=0.0 upper=0.05 effort=50000 velocity=0.1
- added joint l_index_3_shifter: type prismatic, parent l_hand_index_3_shifter, child l_hand_index_3, origin xyz=0.0 0.0 0.0 rpy=0.0 0.0 0.0, axis 0.0 0.0 -1.0, limit lower=0.0 upper=0.05 effort=50000 velocity=0.1
- added joint l_middle_1_shifter: type prismatic, parent l_hand_middle_1, child l_hand_middle_1_shifter, origin xyz=-1.3550151000546462e-07 -0.0014995238274964628 -0.03000020325318492 rpy=-0.0018721728628663644 0 2.576685250299645e-07, axis 0.0 0.0 -1.0, limit lower=0.0 upper=0.05 effort=50000 velocity=0.1
- added joint l_middle_2_shifter: type prismatic, parent l_hand_middle_2_shifter, child l_hand_middle_2, origin xyz=0.0 0.0 0.0 rpy=0.0 0.0 0.0, axis 0.0 0.0 -1.0, limit lower=0.0 upper=0.05 effort=50000 velocity=0.1
- added joint l_pinkie_1_shifter: type prismatic, parent l_hand_pinkie_1, child l_hand_pinkie_1_shifter, origin xyz=0 -0.0014997508602252463 -0.025000232410908152 rpy=3.5631170772755025e-05 -5.94559868174076e-07 -5.245059638522189e-07, axis 0.0 0.0 -1.0, limit lower=0.0 upper=0.05 effort=50000 velocity=0.1
- added joint l_pinkie_2_shifter: type prismatic, parent l_hand_pinkie_2_shifter, child l_hand_pinkie_2, origin xyz=0.0 0.0 0.0 rpy=0.0 0.0 0.0, axis 0.0 0.0 -1.0, limit lower=0.0 upper=0.05 effort=50000 velocity=0.1
- added joint l_ring_1_shifter: type prismatic, parent l_hand_ring_1, child l_hand_ring_1_shifter, origin xyz=0 -0.0014999206015293143 -0.03000056411131863 rpy=0 0 0, axis 0.0 0.0 -1.0, limit lower=0.0 upper=0.05 effort=50000 velocity=0.1
- added joint l_ring_2_shifter: type prismatic, parent l_hand_ring_2_shifter, child l_hand_ring_2, origin xyz=0.0 0.0 0.0 rpy=0.0 0.0 0.0, axis 0.0 0.0 -1.0, limit lower=0.0 upper=0.05 effort=50000 velocity=0.1
- joint l_index_dist: child l_hand_index_3 -> l_hand_index_3_shifter; origin xyz=0 -0.0015006327879180659 -0.02999922319857601 rpy=0 0 0 -> xyz=0.0 0.0 0.0 rpy=0 0 0; parent l_hand_index_2 -> l_hand_index_2_shifter
- joint l_middle_dist: child l_hand_middle_2 -> l_hand_middle_2_shifter; origin xyz=-1.3550151000546462e-07 -0.0014995238274964628 -0.03000020325318492 rpy=-0.0018721728628663644 0 2.576685250299645e-07 -> xyz=0 0 0 rpy=0 0 0; parent l_hand_middle_1 -> l_hand_middle_1_shifter
- joint l_pinkie_dist: child l_hand_pinkie_2 -> l_hand_pinkie_2_shifter; origin xyz=0 -0.0014997508602252463 -0.025000232410908152 rpy=3.5631170772755025e-05 -5.94559868174076e-07 -5.245059638522189e-07 -> xyz=0.0 0.0 0.0 rpy=0.0 0.0 0.0; parent l_hand_pinkie_1 -> l_hand_pinkie_1_shifter
- joint l_ring_dist: child l_hand_ring_2 -> l_hand_ring_2_shifter; origin xyz=0 -0.0014999206015293143 -0.03000056411131863 rpy=0 0 0 -> xyz=0 0 0 rpy=0 0 0; parent l_hand_ring_1 -> l_hand_ring_1_shifter

Commit message: Add fake joints required to study fingers length (continued)

File: urdf/ergoCub/robots/handMK5GazeboV1/model.urdf (robot description, URDF)
Before this commit: robot ergoCub, 25 links, 24 joints
Links:
- removed link l_hand_thumb_2_down_shifter
- removed link l_hand_thumb_2_up_shifter
- added link l_hand_thumb_2_base_shifter, mass 0.1
- added link l_hand_thumb_2_shifter, mass 0.1
Joints:
- removed joint l_thumb_down_shifter
- removed joint l_thumb_shifter_coupled
- added joint l_thumb_2_base_shifter: type prismatic, parent l_hand_thumb_1_pivot, child l_hand_thumb_2_base_shifter, origin xyz= 0.0343950383  0.0313018091 -0.0044737301 rpy=3.0543263593 0.1745316748 0.6632251552, axis -1.0 0.0 0.0, limit lower=0.0 upper=0.03 effort=50000 velocity=0.1
- added joint l_thumb_2_shifter: type prismatic, parent l_hand_thumb_2, child l_hand_thumb_2_shifter, origin xyz=0.01999951842714734 -0.0014995220956423305 4.0850220001109605e-07 rpy=0.0 0.0 0.0, axis 1.0 0.0 0.0, limit lower=0.0 upper=0.03 effort=50000 velocity=0.1
- joint l_thumb_dist: parent l_hand_thumb_2_up_shifter -> l_hand_thumb_2_shifter
- joint l_thumb_prox: parent l_hand_thumb_2_down_shifter -> l_hand_thumb_2_base_shifter

Commit message: Add fake joints required to study fingers length (continued)

File: urdf/ergoCub/robots/handMK5GazeboV1/model.urdf (robot description, URDF)
Before this commit: robot ergoCub, 25 links, 24 joints
Links:
- added link l_hand_thumb_3_shifter, mass 0.1
Joints:
- added joint l_thumb_3_shifter: type prismatic, parent l_hand_thumb_3_shifter, child l_hand_thumb_3, origin xyz=0.0 0.0 0.0 rpy=0.0 0.0 0.0, axis 1.0 0.0 0.0, limit lower=0.0 upper=0.05 effort=50000 velocity=0.1
- joint l_thumb_2_shifter: limit lower=0.0 upper=0.03 effort=50000 velocity=0.1 -> lower=0.0 upper=0.05 effort=50000 velocity=0.1
- joint l_thumb_dist: child l_hand_thumb_3 -> l_hand_thumb_3_shifter

Commit message: Extend the thumb adduction to -10.0 after the latest changes from iCubTech
The thumb now inherits the same limits of the index/middle, moreover the length of the proximal phalanx is also the same as that of the index/middle

File: urdf/ergoCub/robots/handMK5GazeboV1/model.urdf (robot description, URDF)
Before this commit: robot ergoCub, 26 links, 25 joints
Links:
- added link l_hand_thumb_2_offset, mass 0.1
Joints:
- added joint l_thumb_2_offset: type prismatic, parent l_hand_thumb_2, child l_hand_thumb_2_offset, origin xyz=0.02999951842714734 -0.0014995220956423305 4.0850220001109605e-07 rpy=0.0 0.0 0.0, axis 1.0 0.0 0.0, limit lower=0.0 upper=0.0 effort=50000 velocity=0.1
- joint l_thumb_2_shifter: origin xyz=0.01999951842714734 -0.0014995220956423305 4.0850220001109605e-07 rpy=0.0 0.0 0.0 -> xyz=0.0 0.0 0.0 rpy=0.0 0.0 0.0; parent l_hand_thumb_2 -> l_hand_thumb_2_offset
- joint l_thumb_add: limit lower=0.0 upper=3.14 effort=50000 velocity=120.0 -> lower=-0.26 upper=3.14 effort=50000 velocity=120.0
